File: vibe.sch (KiCad schematic (older format))
At the start: 6 parts, among them Q1 Q_NMOS_GSD

Commit message: i2
Parts:
- VS1: footprint (none) -> MyKicadLib:ViSe
Changed lines of the file:
@@
 F 0 "VS1" H 1300 3300 60  0000 C CNN
 F 1 "VIBESENS" H 2000 3300 60  0000 C CNN
-F 2 "" H 1800 3550 60  0001 C CNN
+F 2 "MyKicadLib:ViSe" H 1800 3550 60  0001 C CNN
 F 3 "" H 1800 3550 60  0001 C CNN
 	1    1650 3300
